File: pcb/3V3Digital.kicad_sch (KiCad schematic)
At the start: 4 parts, among them IC9 ADPL42002ARDZ-3.3-R7

Commit message: latest updates to schematic, changed to continuous ground
Parts:
- C65, C66, C67: footprint (none) -> Capacitor_SMD:C_0805_2012Metric
- IC9: footprint SOIC127P600X175-9N -> ADPL42002ARDZ-3.3-R7:SOIC127P600X175-9N
Changed lines of the file:
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@@
 			)
 		)
-		(property "Footprint" ""
+		(property "Footprint" "Capacitor_SMD:C_0805_2012Metric"
 			(at 97.79 88.9 0)
 			(effects
@@
 			)
 		)
-		(property "Footprint" ""
+		(property "Footprint" "Capacitor_SMD:C_0805_2012Metric"
 			(at 161.29 88.9 0)
 			(effects
@@
 			)
 		)
-		(property "Footprint" ""
+		(property "Footprint" "Capacitor_SMD:C_0805_2012Metric"
 			(at 134.62 109.22 0)
 			(effects
@@
 			)
 		)
-		(property "Footprint" "SOIC127P600X175-9N"
+		(property "Footprint" "ADPL42002ARDZ-3.3-R7:SOIC127P600X175-9N"
 			(at 144.78 178.74 0)
 			(effects
