File: pcb/5VRegulator.kicad_sch (KiCad schematic)
At the start: 13 parts

Commit message: latest updates to schematic, changed to continuous ground
Parts:
- C51, C52, C53, C54, C56, C57, C58: footprint (none) -> Capacitor_SMD:C_0805_2012Metric
- IC17: renamed from IC?; footprint SOP65P490X110-13N -> LT3045EMSE#PBF:SOP65P490X110-13N
- R48, R49, R50, R51, R52: footprint (none) -> Resistor_SMD:R_0805_2012Metric
Changed lines of the file:
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@@
 		(dnp no)
 		(fields_autoplaced yes)
-		(property "Reference" "#PWR?"
+		(property "Reference" "#PWR0185"
 			(at 121.92 100.33 0)
 			(effects
@@
 			(project "pcb"
 				(path "/0eb23f11-7b6a-445b-9941-73800592c9c0/a374f7f9-840e-4f0c-b221-b48771a4edc6/3c6e45af-922a-4a02-b622-bda7ee6aa402/38f3ac9c-af0f-47be-bfc0-e866c2baa60e"
-					(reference "#PWR?")
+					(reference "#PWR0185")
 					(unit 1)
 				)
@@
 		(dnp no)
 		(fields_autoplaced yes)
-		(property "Reference" "IC?"
+		(property "Reference" "IC17"
 			(at 119.38 49.53 0)
 			(effects
@@
 			)
 		)
-		(property "Footprint" "SOP65P490X110-13N"
+		(property "Footprint" "LT3045EMSE#PBF:SOP65P490X110-13N"
 			(at 130.81 152.07 0)
 			(effects
@@
 			(project "pcb"
 				(path "/0eb23f11-7b6a-445b-9941-73800592c9c0/a374f7f9-840e-4f0c-b221-b48771a4edc6/3c6e45af-922a-4a02-b622-bda7ee6aa402/38f3ac9c-af0f-47be-bfc0-e866c2baa60e"
-					(reference "IC?")
+					(reference "IC17")
 					(unit 1)
 				)
@@
 			)
 		)
-		(property "Footprint" ""
+		(property "Footprint" "Capacitor_SMD:C_0805_2012Metric"
 			(at 140.97 83.82 0)
 			(effects
@@
 			)
 		)
-		(property "Footprint" ""
+		(property "Footprint" "Resistor_SMD:R_0805_2012Metric"
 			(at 140.97 74.422 90)
 			(effects
@@
 		(dnp no)
 		(fields_autoplaced yes)
-		(property "Reference" "#PWR?"
+		(property "Reference" "#PWR0183"
 			(at 57.15 74.93 0)
 			(effects
@@
 			(project "pcb"
 				(path "/0eb23f11-7b6a-445b-9941-73800592c9c0/a374f7f9-840e-4f0c-b221-b48771a4edc6/3c6e45af-922a-4a02-b622-bda7ee6aa402/38f3ac9c-af0f-47be-bfc0-e866c2baa60e"
-					(reference "#PWR?")
+					(reference "#PWR0183")
 					(unit 1)
 				)
@@
 			)
 		)
-		(property "Footprint" ""
+		(property "Footprint" "Capacitor_SMD:C_0805_2012Metric"
 			(at 76.2 64.77 0)
 			(effects
@@
 			)
 		)
-		(property "Footprint" ""
+		(property "Footprint" "Resistor_SMD:R_0805_2012Metric"
 			(at 97.79 69.342 90)
 			(effects
@@
 			)
 		)
-		(property "Footprint" ""
+		(property "Footprint" "Resistor_SMD:R_0805_2012Metric"
 			(at 102.362 87.63 90)
 			(effects
@@
 			)
 		)
-		(property "Footprint" ""
+		(property "Footprint" "Resistor_SMD:R_0805_2012Metric"
 			(at 154.432 80.01 90)
 			(effects
@@
 			)
 		)
-		(property "Footprint" ""
+		(property "Footprint" "Capacitor_SMD:C_0805_2012Metric"
 			(at 140.97 64.77 0)
 			(effects
@@
 			)
 		)
-		(property "Footprint" ""
+		(property "Footprint" "Capacitor_SMD:C_0805_2012Metric"
 			(at 57.15 62.23 0)
 			(effects
@@
 		(dnp no)
 		(fields_autoplaced yes)
-		(property "Reference" "#PWR?"
+		(property "Reference" "#PWR0184"
 			(at 149.86 85.09 0)
 			(effects
@@
 			(project "pcb"
 				(path "/0eb23f11-7b6a-445b-9941-73800592c9c0/a374f7f9-840e-4f0c-b221-b48771a4edc6/3c6e45af-922a-4a02-b622-bda7ee6aa402/38f3ac9c-af0f-47be-bfc0-e866c2baa60e"
-					(reference "#PWR?")
+					(reference "#PWR0184")
 					(unit 1)
 				)
@@
 			)
 		)
-		(property "Footprint" ""
+		(property "Footprint" "Capacitor_SMD:C_0805_2012Metric"
 			(at 165.1 80.01 0)
 			(effects
@@
 			)
 		)
-		(property "Footprint" ""
+		(property "Footprint" "Capacitor_SMD:C_0805_2012Metric"
 			(at 83.82 67.31 0)
 			(effects
@@
 			)
 		)
-		(property "Footprint" ""
+		(property "Footprint" "Resistor_SMD:R_0805_2012Metric"
 			(at 154.432 68.58 90)
 			(effects
@@
 			)
 		)
-		(property "Footprint" ""
+		(property "Footprint" "Capacitor_SMD:C_0805_2012Metric"
 			(at 67.31 62.23 0)
 			(effects
