File: pcb/AMP_AND_OUT.kicad_sch (KiCad schematic)
At the start: 12 parts, among them IC3 TPA6120A2DWPR, J1 SJ3-35083C-TR

Commit message: latest updates to schematic, changed to continuous ground
Parts:
- C81, C82, C83, C84: footprint (none) -> Capacitor_SMD:C_0805_2012Metric
- IC3: footprint SOIC127P1040X275-21N -> TPA6120A2DWPR:SOIC127P1040X275-21N
- J1: footprint SJ335083CTR -> SJ3-35083C-TR:SJ335083CTR
- R66, R67, R68, R69, R70, R71: footprint (none) -> Resistor_SMD:R_0805_2012Metric
Changed lines of the file:
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@@
 			)
 		)
-		(property "Footprint" ""
+		(property "Footprint" "Capacitor_SMD:C_0805_2012Metric"
 			(at 97.79 105.41 0)
 			(effects
@@
 			)
 		)
-		(property "Footprint" "SOIC127P1040X275-21N"
+		(property "Footprint" "TPA6120A2DWPR:SOIC127P1040X275-21N"
 			(at 69.85 190.17 0)
 			(effects
@@
 			)
 		)
-		(property "Footprint" ""
+		(property "Footprint" "Capacitor_SMD:C_0805_2012Metric"
 			(at 97.79 135.89 0)
 			(effects
@@
 			)
 		)
-		(property "Footprint" ""
+		(property "Footprint" "Resistor_SMD:R_0805_2012Metric"
 			(at 144.78 51.308 90)
 			(effects
@@
 			)
 		)
-		(property "Footprint" ""
+		(property "Footprint" "Resistor_SMD:R_0805_2012Metric"
 			(at 103.632 41.91 90)
 			(effects
@@
 			)
 		)
-		(property "Footprint" "SOIC127P1040X275-21N"
+		(property "Footprint" "TPA6120A2DWPR:SOIC127P1040X275-21N"
 			(at 132.08 183.82 0)
 			(effects
@@
 			)
 		)
-		(property "Footprint" ""
+		(property "Footprint" "Resistor_SMD:R_0805_2012Metric"
 			(at 144.78 83.058 90)
 			(effects
@@
 			)
 		)
-		(property "Footprint" "SOIC127P1040X275-21N"
+		(property "Footprint" "TPA6120A2DWPR:SOIC127P1040X275-21N"
 			(at 95.25 130.48 0)
 			(effects
@@
 			)
 		)
-		(property "Footprint" ""
+		(property "Footprint" "Capacitor_SMD:C_0805_2012Metric"
 			(at 106.68 135.89 0)
 			(effects
@@
 			)
 		)
-		(property "Footprint" "SOIC127P1040X275-21N"
+		(property "Footprint" "TPA6120A2DWPR:SOIC127P1040X275-21N"
 			(at 99.06 152.07 0)
 			(effects
@@
 			)
 		)
-		(property "Footprint" ""
+		(property "Footprint" "Resistor_SMD:R_0805_2012Metric"
 			(at 121.92 93.218 90)
 			(effects
@@
 			)
 		)
-		(property "Footprint" "SJ335083CTR"
+		(property "Footprint" "SJ3-35083C-TR:SJ335083CTR"
 			(at 205.74 159.69 0)
 			(effects
@@
 			)
 		)
-		(property "Footprint" ""
+		(property "Footprint" "Resistor_SMD:R_0805_2012Metric"
 			(at 121.92 61.468 90)
 			(effects
@@
 			)
 		)
-		(property "Footprint" ""
+		(property "Footprint" "Capacitor_SMD:C_0805_2012Metric"
 			(at 106.68 105.41 0)
 			(effects
@@
 			)
 		)
-		(property "Footprint" ""
+		(property "Footprint" "Resistor_SMD:R_0805_2012Metric"
 			(at 103.632 73.66 90)
 			(effects
