File: pcb/Charging.kicad_sch (KiCad schematic)
At the start: 27 parts, among them IC2 TPD4E1U06DBVR, IC6 BQ25883RGER, IC7 TUSB320LAIRWBR, J4 632723300011

Commit message: latest updates to schematic, changed to continuous ground
Parts:
- added R81: 5.23k, Resistor_SMD:R_0805_2012Metric, symbol Device:R
- added R82: 30.1k, Resistor_SMD:R_0805_2012Metric, symbol Device:R
- added TP5: VC2, TestPoint:TestPoint_Pad_3.0x3.0mm, symbol Connector:TestPoint
- C37, C38, C39, C40, C41, C42, C43, C44, C45, C46, C47: footprint (none) -> Capacitor_SMD:C_0805_2012Metric
- D1, D2: footprint SOD123W -> PTVS13VS1UR:SOD123W
- D3: footprint (none) -> LED_SMD:LED_0805_2012Metric
- IC2: footprint SOT95P280X145-6N -> TPD4E1U06DBVR:SOT95P280X145-6N
- IC6: footprint QFN50P400X400X100-25N-D -> BQ25883RGER:QFN50P400X400X100-25N-D
- IC7: footprint RWB0012A -> TUSB320LAIRWBR:RWB0012A
- J4: footprint 632723300011 -> 632723300011:632723300011
- L1: footprint (none) -> Inductor_SMD:L_0805_2012Metric
- R36, R37, R38, R42, R43, R44, R62: footprint (none) -> Resistor_SMD:R_0805_2012Metric
- RT1: value 103AT-2 -> 10K; footprint 103AT2 -> 103AT-2:103AT2
Connections:
- net GND: now also R82.2
- net at C45.1, C46.1, IC6.23 (VBUS)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: now also TP5.1
- net REGN: now reaches C41.1, IC6.11 (REGN)
- net REGN: now also R81.1
- net at IC6.7 (TS), RT1.1: now also R81.2, R82.1
Other:
- moved on the sheet: C41, L1, RT1
