File: pcb/InvertingRegulator.kicad_sch (KiCad schematic)
At the start: 7 parts, among them IC8 LM27761DSGT

Commit message: latest updates to schematic, changed to continuous ground
Parts:
- C48, C49, C50: footprint (none) -> Capacitor_SMD:C_0805_2012Metric
- IC8: footprint SON50P200X200X80-9N -> LM27761DSGT:SON50P200X200X80-9N
- R45, R46, R47: footprint (none) -> Resistor_SMD:R_0805_2012Metric
Changed lines of the file:
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@@
 			)
 		)
-		(property "Footprint" ""
+		(property "Footprint" "Capacitor_SMD:C_0805_2012Metric"
 			(at 91.44 74.93 0)
 			(effects
@@
 			)
 		)
-		(property "Footprint" ""
+		(property "Footprint" "Capacitor_SMD:C_0805_2012Metric"
 			(at 142.24 86.36 0)
 			(effects
@@
 			)
 		)
-		(property "Footprint" "SON50P200X200X80-9N"
+		(property "Footprint" "LM27761DSGT:SON50P200X200X80-9N"
 			(at 137.16 164.77 0)
 			(effects
@@
 			)
 		)
-		(property "Footprint" ""
+		(property "Footprint" "Resistor_SMD:R_0805_2012Metric"
 			(at 148.082 86.36 90)
 			(effects
@@
 			)
 		)
-		(property "Footprint" ""
+		(property "Footprint" "Resistor_SMD:R_0805_2012Metric"
 			(at 148.082 74.93 90)
 			(effects
@@
 			)
 		)
-		(property "Footprint" ""
+		(property "Footprint" "Capacitor_SMD:C_0805_2012Metric"
 			(at 106.68 81.28 0)
 			(effects
@@
 			)
 		)
-		(property "Footprint" ""
+		(property "Footprint" "Resistor_SMD:R_0805_2012Metric"
 			(at 104.14 70.612 90)
 			(effects
