File: pcb/Peripherals.kicad_sch (KiCad schematic)
At the start: 16 parts, among them SW2 SW_Push, SW3 SW_Push, SW4 SW_Nidec_CAS-120A1

Commit message: latest updates to schematic, changed to continuous ground
Parts:
- J3: renamed from J?; footprint 214450577 -> 2-1445057-7:214450577
- J5: renamed from J?; footprint HTSW10209GS -> HTSW-102-09-G-S:HTSW10209GS
- R1, R2, R3: footprint (none) -> Resistor_SMD:R_0805_2012Metric
- R4, R5, R6, R7: renamed from R?; footprint (none) -> Resistor_SMD:R_0805_2012Metric
- SW2, SW3: footprint (none) -> Button_Switch_SMD:SW_Push_1P1T-MP_NO_Horizontal_Alps_SKRTLAE010
- SW5, SW6, SW7, SW8: renamed from SW?; footprint (none) -> Button_Switch_SMD:SW_Push_1P1T-MP_NO_Horizontal_Alps_SKRTLAE010
Connections:
- net GNDD renamed GND
