File: pcb/Regulation.kicad_sch (KiCad schematic)
At the start: 0 parts

Commit message: latest updates to schematic, changed to continuous ground
Parts:
- added TP10, TP6, TP7, TP8, TP9: VC2, TestPoint:TestPoint_Pad_3.0x3.0mm, symbol Connector:TestPoint
Connections:
- net +5V: now also TP7.1
- net -5V: now also TP6.1
- net 3V3A: now also TP8.1
- net 3V3D: now also TP10.1
- net 3V3DAC: now also TP9.1
