File: pcb/untitled.kicad_sch (KiCad schematic)
At the start: 14 parts, among them IC1 ES9038Q2M, U5 LMK6CE

Commit message: latest updates to schematic, changed to continuous ground
Parts:
- C100, C101, C102, C103, C15, C16, C69, C98, C99: footprint (none) -> Capacitor_SMD:C_0805_2012Metric
- IC1: footprint QFN40P300X500X80-31N-D -> ES9038Q2M:QFN40P300X500X80-31N-D
- R40, R79, R80: footprint (none) -> Resistor_SMD:R_0805_2012Metric
- U5: footprint (none) -> BAW:DLF0004A
Changed lines of the file:
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@@
 			)
 		)
-		(property "Footprint" ""
+		(property "Footprint" "Capacitor_SMD:C_0805_2012Metric"
 			(at 96.52 64.77 0)
 			(effects
@@
 			)
 		)
-		(property "Footprint" ""
+		(property "Footprint" "Capacitor_SMD:C_0805_2012Metric"
 			(at 58.42 62.23 0)
 			(effects
@@
 			)
 		)
-		(property "Footprint" ""
+		(property "Footprint" "BAW:DLF0004A"
 			(at 38.1 130.81 0)
 			(effects
@@
 			)
 		)
-		(property "Footprint" ""
+		(property "Footprint" "Resistor_SMD:R_0805_2012Metric"
 			(at 82.042 38.1 90)
 			(effects
@@
 			)
 		)
-		(property "Footprint" ""
+		(property "Footprint" "Capacitor_SMD:C_0805_2012Metric"
 			(at 87.63 43.18 0)
 			(effects
@@
 			)
 		)
-		(property "Footprint" ""
+		(property "Footprint" "Capacitor_SMD:C_0805_2012Metric"
 			(at 38.1 62.23 0)
 			(effects
@@
 			)
 		)
-		(property "Footprint" ""
+		(property "Footprint" "Resistor_SMD:R_0805_2012Metric"
 			(at 22.352 121.92 90)
 			(effects
@@
 			)
 		)
-		(property "Footprint" ""
+		(property "Footprint" "Capacitor_SMD:C_0805_2012Metric"
 			(at 105.41 64.77 0)
 			(effects
@@
 			)
 		)
-		(property "Footprint" "QFN40P300X500X80-31N-D"
+		(property "Footprint" "ES9038Q2M:QFN40P300X500X80-31N-D"
 			(at 66.04 16.84 0)
 			(effects
@@
 			)
 		)
-		(property "Footprint" ""
+		(property "Footprint" "Capacitor_SMD:C_0805_2012Metric"
 			(at 41.91 118.11 0)
 			(effects
@@
 			)
 		)
-		(property "Footprint" ""
+		(property "Footprint" "Resistor_SMD:R_0805_2012Metric"
 			(at 74.422 38.1 90)
 			(effects
@@
 			)
 		)
-		(property "Footprint" ""
+		(property "Footprint" "Capacitor_SMD:C_0805_2012Metric"
 			(at 49.53 62.23 0)
 			(effects
@@
 			)
 		)
-		(property "Footprint" ""
+		(property "Footprint" "Capacitor_SMD:C_0805_2012Metric"
 			(at 72.39 43.18 0)
 			(effects
@@
 		(on_board yes)
 		(dnp no)
-		(property "Reference" "#PWR?"
+		(property "Reference" "#PWR0114"
 			(at 25.4 54.61 0)
 			(effects
@@
 			(project "pcb"
 				(path "/0eb23f11-7b6a-445b-9941-73800592c9c0/cb4f690f-8ee1-423e-9713-b2411228fffc"
-					(reference "#PWR?")
+					(reference "#PWR0114")
 					(unit 1)
 				)
@@
 			)
 		)
-		(property "Footprint" ""
+		(property "Footprint" "Capacitor_SMD:C_0805_2012Metric"
 			(at 29.21 62.23 0)
 			(effects
